File: spi_pcb.kicad_pcb (KiCad board)
At the start: 2 copper layers, 65 x 56 mm, 20 parts, among them J1 GPIO, J2 PWR, U1 imported:LMZ23605TZ

Commit message: Split feedback resistors into available values.
Parts:
- added Rfb1: 1k, Resistor_SMD:R_0603_1608Metric, F.Cu at (126.3, 82.1)
- Rfb2: renamed from R2; value 1.05k -> 51
- moved Rfb2 0.17 mm to (128.1, 83.7)
- moved R1 0.05 mm to (124.6, 83.7)
Connections:
- Rfb2 pad 1: Net-(U1-FB) -> Net-(Rfb1-Pad2)
Routing:
- net Net-(U1-FB): track 7.36 -> 5.05 mm
- net Net-(Rfb1-Pad2): track 0.00 -> 1.66 mm
- net GND: vias 35 -> 32
Changed lines of the file:
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@@
 	(net 41 "Net-(SPI2-Pin_3)")
 	(net 42 "Net-(SPI2-Pin_5)")
+	(net 43 "Net-(Rfb1-Pad2)")
 	(footprint "imported:EEFCX0J101R"
 		(layer "F.Cu")
@@
 	(footprint "Resistor_SMD:R_0603_1608Metric"
 		(layer "F.Cu")
-		(at 127.9425 83.755)
+		(at 128.1 83.7)
 		(descr "Resistor SMD 0603 (1608 Metric), square (rectangular) end terminal, IPC_7351 nominal, (Body size source: IPC-SM-782 page 72, https://www.pcb-3d.com/wordpress/wp-content/uploads/ipc-sm-782a_amendment_1_and_2.pdf), generated with kicad-footprint-generator")
 		(tags "resistor")
-		(property "Reference" "R2"
+		(property "Reference" "Rfb2"
 			(at 0 -1.43 0)
 			(layer "F.SilkS")
@@
 			)
 		)
-		(property "Value" "1.05k"
+		(property "Value" "51"
 			(at 0 1.43 0)
 			(layer "F.Fab")
@@
 			(layers "F.Cu" "F.Mask" "F.Paste")
 			(roundrect_rratio 0.25)
-			(net 30 "Net-(U1-FB)")
+			(net 43 "Net-(Rfb1-Pad2)")
 			(pintype "passive")
 		)
@@
 	(footprint "Resistor_SMD:R_0603_1608Metric"
 		(layer "F.Cu")
-		(at 124.6175 83.755)
+		(at 124.6175 83.7)
 		(descr "Resistor SMD 0603 (1608 Metric), square (rectangular) end terminal, IPC_7351 nominal, (Body size source: IPC-SM-782 page 72, https://www.pcb-3d.com/wordpress/wp-content/uploads/ipc-sm-782a_amendment_1_and_2.pdf), generated with kicad-footprint-generator")
 		(tags "resistor")
@@
 		)
 	)
+	(footprint "Resistor_SMD:R_0603_1608Metric"
+		(layer "F.Cu")
+		(at 126.3 82.1)
+		(descr "Resistor SMD 0603 (1608 Metric), square (rectangular) end terminal, IPC_7351 nominal, (Body size source: IPC-SM-782 page 72, https://www.pcb-3d.com/wordpress/wp-content/uploads/ipc-sm-782a_amendment_1_and_2.pdf), generated with kicad-footprint-generator")
+		(tags "resistor")
+		(property "Reference" "Rfb1"
+			(at 0 -1.43 0)
+			(layer "F.SilkS")
+			(effects
+				(font
+					(size 1 1)
+					(thickness 0.15)
+				)
+			)
+		)
+		(property "Value" "1k"
+			(at 0 1.43 0)
+			(layer "F.Fab")
+			(effects
+				(font
+					(size 1 1)
+					(thickness 0.15)
+				)
+			)
+		)
+		(property "Datasheet" "https://fr.farnell.com/multicomp-pro/mcwr06x1051ftl/resist-1k05-1-0-1w-couche-epaisse/dp/2447273"
+			(at 0 0 0)
+			(unlocked yes)
+			(layer "F.Fab")
+			(hide yes)
+			(effects
+				(font
+					(size 1.27 1.27)
+					(thickness 0.15)
+				)
+			)
+		)
+		(property "Description" "Resistor"
+			(at 0 0 0)
+			(unlocked yes)
+			(layer "F.Fab")
+			(hide yes)
+			(effects
+				(font
+					(size 1.27 1.27)
+					(thickness 0.15)
+				)
+			)
+		)
+		(property ki_fp_filters "R_*")
+		(sheetname "/")
+		(sheetfile "spi_pcb.kicad_sch")
+		(attr smd)
+		(fp_line
+			(start -0.237258 -0.5225)
+			(end 0.237258 -0.5225)
+			(stroke
+				(width 0.12)
+				(type solid)
+			)
+			(layer "F.SilkS")
+		)
+		(fp_line
+			(start -0.237258 0.5225)
+			(end 0.237258 0.5225)
+			(stroke
+				(width 0.12)
+				(type solid)
+			)
+			(layer "F.SilkS")
+		)
+		(fp_line
+			(start -1.48 -0.73)
+			(end 1.48 -0.73)
+			(stroke
+				(width 0.05)
+				(type solid)
+			)
+			(layer "F.CrtYd")
+		)
+		(fp_line
+			(start -1.48 0.73)
+			(end -1.48 -0.73)
+			(stroke
+				(width 0.05)
+				(type solid)
+			)
+			(layer "F.CrtYd")
+		)
+		(fp_line
+			(start 1.48 -0.73)
+			(end 1.48 0.73)
+			(stroke
+				(width 0.05)
+				(type solid)
+			)
+			(layer "F.CrtYd")
+		)
+		(fp_line
+			(start 1.48 0.73)
+			(end -1.48 0.73)
+			(stroke
+				(width 0.05)
+				(type solid)
+			)
+			(layer "F.CrtYd")
+		)
+		(fp_line
+			(start -0.8 -0.4125)
+			(end 0.8 -0.4125)
+			(stroke
+				(width 0.1)
+				(type solid)
+			)
+			(layer "F.Fab")
+		)
+		(fp_line
+			(start -0.8 0.4125)
+			(end -0.8 -0.4125)
+			(stroke
+				(width 0.1)
+				(type solid)
+			)
+			(layer "F.Fab")
+		)
+		(fp_line
+			(start 0.8 -0.4125)
+			(end 0.8 0.4125)
+			(stroke
+				(width 0.1)
+				(type solid)
+			)
+			(layer "F.Fab")
+		)
+		(fp_line
+			(start 0.8 0.4125)
+			(end -0.8 0.4125)
+			(stroke
+				(width 0.1)
+				(type solid)
+			)
+			(layer "F.Fab")
+		)
+		(fp_text user "${REFERENCE}"
+			(at 0 0 0)
+			(layer "F.Fab")
+			(effects
+				(font
+					(size 0.4 0.4)
+					(thickness 0.06)
+				)
+			)
+		)
+		(pad "1" smd roundrect
+			(at -0.825 0)
+			(size 0.8 0.95)
+			(layers "F.Cu" "F.Mask" "F.Paste")
+			(roundrect_rratio 0.25)
+			(net 30 "Net-(U1-FB)")
+			(pintype "passive")
+		)
+		(pad "2" smd roundrect
+			(at 0.825 0)
+			(size 0.8 0.95)
+			(layers "F.Cu" "F.Mask" "F.Paste")
+			(roundrect_rratio 0.25)
+			(net 43 "Net-(Rfb1-Pad2)")
+			(pintype "passive")
+		)
+		(embedded_fonts no)
+		(model "${KICAD9_3DMODEL_DIR}/Resistor_SMD.3dshapes/R_0603_1608Metric.wrl"
+			(offset
+				(xyz 0 0 0)
+			)
+			(scale
+				(xyz 1 1 1)
+			)
+			(rotate
+				(xyz 0 0 0)
+			)
+		)
+	)
 	(footprint "Resistor_SMD:R_0402_1005Metric_Pad0.72x0.64mm_HandSolder"
 		(layer "F.Cu")
@@
 	)
 	(via
-		(at 129.4 80.8)
-		(size 1)
-		(drill 0.5)
-		(layers "F.Cu" "B.Cu")
-		(net 1)
-	)
-	(via
 		(at 141.4 52.6)
 		(size 1)
@@
 	)
 	(via
-		(at 125.4 80.8)
-		(size 1)
-		(drill 0.5)
-		(layers "F.Cu" "B.Cu")
-		(net 1)
-	)
-	(via
 		(at 119.9 96.8)
 		(size 1)
@@
 	)
 	(via
-		(at 127.4 80.8)
-		(size 1)
-		(drill 0.5)
-		(layers "F.Cu" "B.Cu")
-		(net 1)
-	)
-	(via
 		(at 158.9 50.8)
 		(size 1)
@@
 	)
 	(segment
-		(start 125.2425 85.63)
+		(start 125.4425 83.7)
+		(end 125.4425 86.805)
+		(width 0.3)
+		(layer "F.Cu")
+		(net 30)
+	)
+	(segment
+		(start 125.4425 86.805)
 		(end 125.2425 87.005)
 		(width 0.3)
@@
 	)
 	(segment
-		(start 125.4425 83.755)
-		(end 125.4425 86.805)
+		(start 125.475 82.1)
+		(end 125.475 83.6675)
 		(width 0.3)
 		(layer "F.Cu")
@@
 	)
 	(segment
-		(start 127.1175 83.755)
-		(end 125.2425 85.63)
+		(start 125.475 83.7225)
+		(end 125.4425 83.755)
 		(width 0.3)
 		(layer "F.Cu")
@@
 	)
 	(segment
-		(start 125.4425 86.805)
-		(end 125.2425 87.005)
+		(start 125.475 83.6675)
+		(end 125.4425 83.7)
 		(width 0.3)
 		(layer "F.Cu")
@@
 		(net 42)
 	)
+	(segment
+		(start 127.125 83.55)
+		(end 127.275 83.7)
+		(width 0.3)
+		(layer "F.Cu")
+		(net 43)
+	)
+	(segment
+		(start 127.125 82.1)
+		(end 127.125 83.55)
+		(width 0.3)
+		(layer "F.Cu")
+		(net 43)
+	)
 	(zone

Commit message: Increased via diameter to allow for wire soldering.
Routing:
- net GND: track 91.7 -> 74.9 mm, vias 32 -> 33
- net +5V: vias 16 -> 14
